File: Relays_and_sensor.kicad_sch (KiCad schematic)
At the start: 0 parts

Commit message: Rain sensor
Parts:
- added C?: 100nF, symbol Device:C
- added J?: Screw_Terminal_01x02, symbol Connector:Screw_Terminal_01x02
- added R?: 6.49k, symbol Device:R
- added R?: 1k, symbol Device:R
Connections:
- new net: J?.1 (Pin_1), R?.2, R?.2
- new net GND: C?.2, J?.2 (Pin_2)
- new net Rain_Sensor: C?.1, R?.1
- new net VDD: R?.1
Changed lines of the file:
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@@
     (comment 2 "Laboratoria")
   )
+  (junction (at 64.77 160.02) (diameter 0) (color 0 0 0 0)
+  )
+  (junction (at 64.77 175.26) (diameter 0) (color 0 0 0 0)
+  )
+  (wire (pts (xy 64.77 153.67) (xy 64.77 160.02))
+    (stroke (width 0) (type default) (color 0 0 0 0))
+  )
+  (wire (pts (xy 64.77 175.26) (xy 64.77 180.34))
+    (stroke (width 0) (type default) (color 0 0 0 0))
+  )
+  (wire (pts (xy 64.77 160.02) (xy 68.58 160.02))
+    (stroke (width 0) (type default) (color 0 0 0 0))
+  )
+  (wire (pts (xy 73.66 180.34) (xy 78.74 180.34))
+    (stroke (width 0) (type default) (color 0 0 0 0))
+  )
+  (wire (pts (xy 64.77 180.34) (xy 71.12 180.34))
+    (stroke (width 0) (type default) (color 0 0 0 0))
+  )
+  (wire (pts (xy 76.2 160.02) (xy 80.01 160.02))
+    (stroke (width 0) (type default) (color 0 0 0 0))
+  )
+  (wire (pts (xy 60.96 175.26) (xy 64.77 175.26))
+    (stroke (width 0) (type default) (color 0 0 0 0))
+  )
+  (wire (pts (xy 64.77 171.45) (xy 64.77 175.26))
+    (stroke (width 0) (type default) (color 0 0 0 0))
+  )
+  (wire (pts (xy 64.77 163.83) (xy 64.77 160.02))
+    (stroke (width 0) (type default) (color 0 0 0 0))
+  )
+  (wire (pts (xy 50.8 175.26) (xy 53.34 175.26))
+    (stroke (width 0) (type default) (color 0 0 0 0))
+  )
+  (global_label "Rain_Sensor" (shape output) (at 64.77 153.67 90) (fields_autoplaced)
+    (effects (font (size 1.27 1.27)) (justify left))
+    (property "Intersheet References" "${INTERSHEET_REFS}" (id 0) (at 64.6906 139.7059 90)
+      (effects (font (size 1.27 1.27)) (justify left) hide)
+    )
+  )
+  (symbol (lib_id "power:VDD") (at 50.8 175.26 90) (unit 1)
+    (in_bom yes) (on_board yes)
+    (property "Reference" "#PWR?" (id 0) (at 54.61 175.26 0)
+      (effects (font (size 1.27 1.27)) hide)
+    )
+    (property "Value" "VDD" (id 1) (at 47.625 172.72 0))
+    (property "Footprint" "" (id 2) (at 50.8 175.26 0)
+      (effects (font (size 1.27 1.27)) hide)
+    )
+    (property "Datasheet" "" (id 3) (at 50.8 175.26 0)
+      (effects (font (size 1.27 1.27)) hide)
+    )
+    (pin "1")
+  )
+  (symbol (lib_id "Device:R") (at 57.15 175.26 90) (unit 1)
+    (in_bom yes) (on_board yes) (fields_autoplaced)
+    (property "Reference" "R?" (id 0) (at 57.15 168.91 90))
+    (property "Value" "6.49k" (id 1) (at 57.15 171.45 90))
+    (property "Footprint" "" (id 2) (at 57.15 177.038 90)
+      (effects (font (size 1.27 1.27)) hide)
+    )
+    (property "Datasheet" "~" (id 3) (at 57.15 175.26 0)
+      (effects (font (size 1.27 1.27)) hide)
+    )
+    (pin "1")
+    (pin "2")
+  )
+  (symbol (lib_id "power:GND") (at 78.74 180.34 90) (unit 1)
+    (in_bom yes) (on_board yes) (fields_autoplaced)
+    (property "Reference" "#PWR?" (id 0) (at 85.09 180.34 0)
+      (effects (font (size 1.27 1.27)) hide)
+    )
+    (property "Value" "GND" (id 1) (at 82.55 180.3399 90)
+      (effects (font (size 1.27 1.27)) (justify right))
+    )
+    (property "Footprint" "" (id 2) (at 78.74 180.34 0)
+      (effects (font (size 1.27 1.27)) hide)
+    )
+    (property "Datasheet" "" (id 3) (at 78.74 180.34 0)
+      (effects (font (size 1.27 1.27)) hide)
+    )
+    (pin "1")
+  )
+  (symbol (lib_id "power:GND") (at 80.01 160.02 90) (unit 1)
+    (in_bom yes) (on_board yes) (fields_autoplaced)
+    (property "Reference" "#PWR?" (id 0) (at 86.36 160.02 0)
+      (effects (font (size 1.27 1.27)) hide)
+    )
+    (property "Value" "GND" (id 1) (at 83.82 160.0199 90)
+      (effects (font (size 1.27 1.27)) (justify right))
+    )
+    (property "Footprint" "" (id 2) (at 80.01 160.02 0)
+      (effects (font (size 1.27 1.27)) hide)
+    )
+    (property "Datasheet" "" (id 3) (at 80.01 160.02 0)
+      (effects (font (size 1.27 1.27)) hide)
+    )
+    (pin "1")
+  )
+  (symbol (lib_id "Device:C") (at 72.39 160.02 90) (unit 1)
+    (in_bom yes) (on_board yes) (fields_autoplaced)
+    (property "Reference" "C?" (id 0) (at 72.39 152.4 90))
+    (property "Value" "100nF" (id 1) (at 72.39 154.94 90))
+    (property "Footprint" "" (id 2) (at 76.2 159.0548 0)
+      (effects (font (size 1.27 1.27)) hide)
+    )
+    (property "Datasheet" "~" (id 3) (at 72.39 160.02 0)
+      (effects (font (size 1.27 1.27)) hide)
+    )
+    (pin "1")
+    (pin "2")
+  )
+  (symbol (lib_id "Device:R") (at 64.77 167.64 0) (unit 1)
+    (in_bom yes) (on_board yes) (fields_autoplaced)
+    (property "Reference" "R?" (id 0) (at 67.31 166.3699 0)
+      (effects (font (size 1.27 1.27)) (justify left))
+    )
+    (property "Value" "1k" (id 1) (at 67.31 168.9099 0)
+      (effects (font (size 1.27 1.27)) (justify left))
+    )
+    (property "Footprint" "" (id 2) (at 62.992 167.64 90)
+      (effects (font (size 1.27 1.27)) hide)
+    )
+    (property "Datasheet" "~" (id 3) (at 64.77 167.64 0)
+      (effects (font (size 1.27 1.27)) hide)
+    )
+    (pin "1")
+    (pin "2")
+  )
+  (symbol (lib_id "Connector:Screw_Terminal_01x02") (at 71.12 175.26 90) (unit 1)
+    (in_bom yes) (on_board yes) (fields_autoplaced)
+    (property "Reference" "J?" (id 0) (at 76.2 173.9899 90)
+      (effects (font (size 1.27 1.27)) (justify right))
+    )
+    (property "Value" "Screw_Terminal_01x02" (id 1) (at 76.2 176.5299 90)
+      (effects (font (size 1.27 1.27)) (justify right))
+    )
+    (property "Footprint" "" (id 2) (at 71.12 175.26 0)
+      (effects (font (size 1.27 1.27)) hide)
+    )
+    (property "Datasheet" "~" (id 3) (at 71.12 175.26 0)
+      (effects (font (size 1.27 1.27)) hide)
+    )
+    (pin "1")
+    (pin "2")
+  )
 )

Commit message: ver 0.1
Parts:
- added D1, D2, D3, D4: 1N4007G, DIOAD1036W78L470D235, symbol 1N4007G:1N4007G
- added J5, J6, J7, J8: Screw_Terminal_01x02, symbol Connector:Screw_Terminal_01x02
- added K1, K2, K3, K4: 1461103-1, symbol Project_lib_symbols_AM:1461103-1
- added Q1, Q2, Q3, Q4: ZTX450, symbol Device:Q_NPN_BCE
- added R23, R24, R27, R28: 220, symbol Device:R
- gave numbers to parts that had none: 4
Connections:
- net GND: now also J5.2 (Pin_2), J6.2 (Pin_2), J7.2 (Pin_2), J8.2 (Pin_2), Q1.3 (E), Q2.3 (E), Q3.3 (E), Q4.3 (E)
- net VDD: now also D1.C, D2.C, D3.C, D4.C, K1.2, K2.2, K3.2, K4.2
- net Rain_Sensor renamed Rain_sensor
- new net: D1.A, K1.1, Q1.2 (C)
- new net: Q1.1 (B), R23.2
- new net: D4.A, K4.1, Q4.2 (C)
- new net: J8.1 (Pin_1), K4.4
- new net: J7.1 (Pin_1), K3.4
- new net: J5.1 (Pin_1), K1.4
- new net: D2.A, K2.1, Q2.2 (C)
- new net: Q2.1 (B), R24.2
- new net: D3.A, K3.1, Q3.2 (C)
- new net: Q4.1 (B), R28.2
- new net: J6.1 (Pin_1), K2.4
- new net: Q3.1 (B), R27.2
- new net 24V: K1.3, K2.3, K3.3, K4.3
- new net Valve_1: R23.1
- new net Valve_2: R27.1
- new net Valve_3: R24.1
- new net Valve_4: R28.1
Other:
- note added: "Rain sensor"
- note added: "Valve relays"
- moved on the sheet: C22, J4, R25, R26

Commit message: Lab 07.11
Parts:
- R25: value 6.49k -> 10k
Connections:
- net 24V renamed +24V
Changed lines of the file:
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@@
+    (stroke (width 0) (type default) (color 0 0 0 0))
+  )
+  (wire (pts (xy 72.39 45.085) (xy 72.39 48.895))
     (stroke (width 0) (type default) (color 0 0 0 0))
   )
@@
     (stroke (width 0) (type default) (color 0 0 0 0))
   )
+  (wire (pts (xy 171.45 45.085) (xy 171.45 50.165))
+    (stroke (width 0) (type default) (color 0 0 0 0))
+  )
   (wire (pts (xy 57.785 154.94) (xy 61.595 154.94))
     (stroke (width 0) (type default) (color 0 0 0 0))
@@
     (stroke (width 0) (type default) (color 0 0 0 0))
   )
+  (wire (pts (xy 171.45 102.235) (xy 176.53 102.235))
+    (stroke (width 0) (type default) (color 0 0 0 0))
+  )
   (wire (pts (xy 43.18 96.52) (xy 52.07 96.52))
     (stroke (width 0) (type default) (color 0 0 0 0))
@@
     (stroke (width 0) (type default) (color 0 0 0 0))
   )
+  (wire (pts (xy 72.39 101.6) (xy 78.105 101.6))
+    (stroke (width 0) (type default) (color 0 0 0 0))
+  )
   (wire (pts (xy 192.405 90.17) (xy 192.405 95.885))
     (stroke (width 0) (type default) (color 0 0 0 0))
@@
     (stroke (width 0) (type default) (color 0 0 0 0))
   )
+  (wire (pts (xy 72.39 96.52) (xy 72.39 101.6))
+    (stroke (width 0) (type default) (color 0 0 0 0))
+  )
   (wire (pts (xy 43.18 81.28) (xy 52.07 81.28))
     (stroke (width 0) (type default) (color 0 0 0 0))
@@
     (stroke (width 0) (type default) (color 0 0 0 0))
   )
+  (wire (pts (xy 72.39 48.895) (xy 76.835 48.895))
+    (stroke (width 0) (type default) (color 0 0 0 0))
+  )
   (polyline (pts (xy 14.605 17.145) (xy 14.605 128.905))
     (stroke (width 0) (type default) (color 0 0 0 0))
@@
     (stroke (width 0) (type default) (color 0 0 0 0))
   )
+  (wire (pts (xy 171.45 96.52) (xy 171.45 102.235))
+    (stroke (width 0) (type default) (color 0 0 0 0))
+  )
   (wire (pts (xy 142.24 45.085) (xy 151.13 45.085))
     (stroke (width 0) (type default) (color 0 0 0 0))
@@
   )
   (wire (pts (xy 151.13 96.52) (xy 151.13 100.965))
+    (stroke (width 0) (type default) (color 0 0 0 0))
+  )
+  (wire (pts (xy 171.45 50.165) (xy 177.165 50.165))
     (stroke (width 0) (type default) (color 0 0 0 0))
   )
@@
     (effects (font (size 2 2)) (justify right bottom))
   )
-  (hierarchical_label "24V" (shape input) (at 171.45 45.085 270)
-    (effects (font (size 1.27 1.27)) (justify right))
-  )
   (hierarchical_label "Valve_2" (shape input) (at 123.825 54.61 180)
     (effects (font (size 1.27 1.27)) (justify right))
@@
     (effects (font (size 1.27 1.27)) (justify right))
   )
-  (hierarchical_label "24V" (shape input) (at 72.39 96.52 270)
-    (effects (font (size 1.27 1.27)) (justify right))
-  )
   (hierarchical_label "Valve_3" (shape input) (at 24.765 106.045 180)
     (effects (font (size 1.27 1.27)) (justify right))
   )
-  (hierarchical_label "24V" (shape input) (at 171.45 96.52 270)
-    (effects (font (size 1.27 1.27)) (justify right))
-  )
   (hierarchical_label "Valve_1" (shape input) (at 24.765 54.61 180)
     (effects (font (size 1.27 1.27)) (justify right))
@@
   (hierarchical_label "Rain_sensor" (shape output) (at 57.785 148.59 90)
     (effects (font (size 1.27 1.27)) (justify left))
-  )
-  (hierarchical_label "24V" (shape input) (at 72.39 45.085 270)
-    (effects (font (size 1.27 1.27)) (justify right))
   )
   (symbol (lib_id "power:VDD") (at 151.13 27.305 0) (unit 1)
@@
     (in_bom yes) (on_board yes) (fields_autoplaced)
     (property "Reference" "R25" (id 0) (at 50.165 163.83 90))
-    (property "Value" "6.49k" (id 1) (at 50.165 166.37 90))
+    (property "Value" "10k" (id 1) (at 50.165 166.37 90))
     (property "Footprint" "" (id 2) (at 50.165 171.958 90)
       (effects (font (size 1.27 1.27)) hide)
@@
     )
     (property "Datasheet" "" (id 3) (at 93.345 44.45 0)
+      (effects (font (size 1.27 1.27)) hide)
+    )
+    (pin "1")
+  )
+  (symbol (lib_id "power:+24V") (at 78.105 101.6 0) (unit 1)
+    (in_bom yes) (on_board yes) (fields_autoplaced)
+    (property "Reference" "#PWR062" (id 0) (at 78.105 105.41 0)
+      (effects (font (size 1.27 1.27)) hide)
+    )
+    (property "Value" "+24V" (id 1) (at 78.105 95.885 0))
+    (property "Footprint" "" (id 2) (at 78.105 101.6 0)
+      (effects (font (size 1.27 1.27)) hide)
+    )
+    (property "Datasheet" "" (id 3) (at 78.105 101.6 0)
       (effects (font (size 1.27 1.27)) hide)
     )
@@
     (pin "2")
   )
+  (symbol (lib_id "power:+24V") (at 176.53 102.235 0) (unit 1)
+    (in_bom yes) (on_board yes) (fields_autoplaced)
+    (property "Reference" "#PWR063" (id 0) (at 176.53 106.045 0)
+      (effects (font (size 1.27 1.27)) hide)
+    )
+    (property "Value" "+24V" (id 1) (at 176.53 96.52 0))
+    (property "Footprint" "" (id 2) (at 176.53 102.235 0)
+      (effects (font (size 1.27 1.27)) hide)
+    )
+    (property "Datasheet" "" (id 3) (at 176.53 102.235 0)
+      (effects (font (size 1.27 1.27)) hide)
+    )
+    (pin "1")
+  )
   (symbol (lib_id "power:GND") (at 151.13 64.135 0) (unit 1)
     (in_bom yes) (on_board yes) (fields_autoplaced)
@@
     (pin "2")
   )
+  (symbol (lib_id "power:+24V") (at 177.165 50.165 0) (unit 1)
+    (in_bom yes) (on_board yes) (fields_autoplaced)
+    (property "Reference" "#PWR064" (id 0) (at 177.165 53.975 0)
+      (effects (font (size 1.27 1.27)) hide)
+    )
+    (property "Value" "+24V" (id 1) (at 177.165 44.45 0))
+    (property "Footprint" "" (id 2) (at 177.165 50.165 0)
+      (effects (font (size 1.27 1.27)) hide)
+    )
+    (property "Datasheet" "" (id 3) (at 177.165 50.165 0)
+      (effects (font (size 1.27 1.27)) hide)
+    )
+    (pin "1")
+  )
   (symbol (lib_id "Connector:Screw_Terminal_01x02") (at 98.425 87.63 0) (unit 1)
     (in_bom yes) (on_board yes) (fields_autoplaced)
@@
       (effects (font (size 1.27 1.27)) hide)
     )
+    (pin "1")
+  )
+  (symbol (lib_id "power:+24V") (at 76.835 48.895 0) (unit 1)
+    (in_bom yes) (on_board yes) (fields_autoplaced)
+    (property "Reference" "#PWR061" (id 0) (at 76.835 52.705 0)
+      (effects (font (size 1.27 1.27)) hide)
+    )
+    (property "Value" "+24V" (id 1) (at 76.835 43.18 0))
+    (property "Footprint" "" (id 2) (at 76.835 48.895 0)
+      (effects (font (size 1.27 1.27)) hide)
+    )
+    (property "Datasheet" "" (id 3) (at 76.835 48.895 0)
+      (effects (font (size 1.27 1.27)) hide)
+    )

Commit message: Isolation
Parts:
- added R29, R30, R31, R5: 220, symbol Device:R
- added U3: LTV-844, Package_DIP:DIP-16_W7.62mm, symbol Isolator:LTV-844
Connections:
- net GND: now also U3.2, U3.4, U3.6, U3.8
- net VDD: now also U3.10, U3.12, U3.14, U3.16
- net Valve_1: now also R29.1; no longer R23.1
- net Valve_2: now also R30.1; no longer R27.1
- net Valve_3: now also R5.1; no longer R24.1
- net Valve_4: now also R31.1; no longer R28.1
- new net: R29.2, U3.1
- new net: R24.1, U3.13
- new net: R5.2, U3.3
- new net: R31.2, U3.7
- new net: R30.2, U3.5
- new net: R28.1, U3.9
- new net: R27.1, U3.11
- new net: R23.1, U3.15
Other:
- moved on the sheet: D1, D2, D3, D4, J5, J6, J7, J8, K1, K2, K3, K4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

Commit message: Rezystory, kondensatory, cewka - footprints
Parts:
- C22: footprint (none) -> Capacitor_SMD:C_0603_1608Metric
- D1, D2, D3, D4: footprint DIOAD1036W78L470D235 -> (none)
- R23, R24, R25, R26, R27, R28, R29, R30, R31, R5: footprint (none) -> Resistor_SMD:R_0603_1608Metric
Changed lines of the file:
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@@
       (effects (font (size 1.27 1.27)) (justify right))
     )
-    (property "Footprint" "DIOAD1036W78L470D235" (id 2) (at 66.04 36.83 0)
+    (property "Footprint" "" (id 2) (at 66.04 36.83 0)
       (effects (font (size 1.27 1.27)) (justify left bottom) hide)
     )
@@
     (property "Reference" "R25" (id 0) (at 50.165 163.83 90))
     (property "Value" "10k" (id 1) (at 50.165 166.37 90))
-    (property "Footprint" "" (id 2) (at 50.165 171.958 90)
+    (property "Footprint" "Resistor_SMD:R_0603_1608Metric" (id 2) (at 50.165 171.958 90)
       (effects (font (size 1.27 1.27)) hide)
     )
@@
     (property "Reference" "R29" (id 0) (at 29.21 43.18 90))
     (property "Value" "220" (id 1) (at 29.21 45.72 90))
-    (property "Footprint" "" (id 2) (at 29.21 50.673 90)
+    (property "Footprint" "Resistor_SMD:R_0603_1608Metric" (id 2) (at 29.21 50.673 90)
       (effects (font (size 1.27 1.27)) hide)
     )
@@
     (property "Reference" "R31" (id 0) (at 153.67 92.71 90))
     (property "Value" "220" (id 1) (at 153.67 95.25 90))
-    (property "Footprint" "" (id 2) (at 153.67 100.203 90)
+    (property "Footprint" "Resistor_SMD:R_0603_1608Metric" (id 2) (at 153.67 100.203 90)
       (effects (font (size 1.27 1.27)) hide)
     )
@@
     (property "Reference" "R5" (id 0) (at 28.575 92.71 90))
     (property "Value" "220" (id 1) (at 28.575 95.25 90))
-    (property "Footprint" "" (id 2) (at 28.575 100.203 90)
+    (property "Footprint" "Resistor_SMD:R_0603_1608Metric" (id 2) (at 28.575 100.203 90)
       (effects (font (size 1.27 1.27)) hide)
     )
@@
       (effects (font (size 1.27 1.27)) (justify right))
     )
-    (property "Footprint" "DIOAD1036W78L470D235" (id 2) (at 66.04 86.36 0)
+    (property "Footprint" "" (id 2) (at 66.04 86.36 0)
       (effects (font (size 1.27 1.27)) (justify left bottom) hide)
     )
@@
     (property "Reference" "R30" (id 0) (at 146.05 43.18 90))
     (property "Value" "220" (id 1) (at 146.05 45.72 90))
-    (property "Footprint" "" (id 2) (at 146.05 50.673 90)
+    (property "Footprint" "Resistor_SMD:R_0603_1608Metric" (id 2) (at 146.05 50.673 90)
       (effects (font (size 1.27 1.27)) hide)
     )
@@
     (property "Reference" "R24" (id 0) (at 59.055 97.79 90))
     (property "Value" "220" (id 1) (at 59.055 100.33 90))
-    (property "Footprint" "" (id 2) (at 59.055 105.283 90)
+    (property "Footprint" "Resistor_SMD:R_0603_1608Metric" (id 2) (at 59.055 105.283 90)
       (effects (font (size 1.27 1.27)) hide)
     )
@@
       (effects (font (size 1.27 1.27)) (justify right))
     )
-    (property "Footprint" "DIOAD1036W78L470D235" (id 2) (at 191.135 36.83 0)
+    (property "Footprint" "" (id 2) (at 191.135 36.83 0)
       (effects (font (size 1.27 1.27)) (justify left bottom) hide)
     )
@@
     (property "Reference" "R28" (id 0) (at 184.15 97.79 90))
     (property "Value" "220" (id 1) (at 184.15 100.33 90))
-    (property "Footprint" "" (id 2) (at 184.15 105.283 90)
+    (property "Footprint" "Resistor_SMD:R_0603_1608Metric" (id 2) (at 184.15 105.283 90)
       (effects (font (size 1.27 1.27)) hide)
     )
@@
       (effects (font (size 1.27 1.27)) (justify right))
     )
-    (property "Footprint" "DIOAD1036W78L470D235" (id 2) (at 191.135 86.36 0)
+    (property "Footprint" "" (id 2) (at 191.135 86.36 0)
       (effects (font (size 1.27 1.27)) (justify left bottom) hide)
     )
@@
     (property "Reference" "C22" (id 0) (at 65.405 147.32 90))
     (property "Value" "100nF" (id 1) (at 65.405 149.86 90))
-    (property "Footprint" "" (id 2) (at 69.215 153.9748 0)
+    (property "Footprint" "Capacitor_SMD:C_0603_1608Metric" (id 2) (at 69.215 153.9748 0)
       (effects (font (size 1.27 1.27)) hide)
     )
@@
       (effects (font (size 1.27 1.27)) (justify left))
     )
-    (property "Footprint" "" (id 2) (at 56.007 162.56 90)
+    (property "Footprint" "Resistor_SMD:R_0603_1608Metric" (id 2) (at 56.007 162.56 90)
       (effects (font (size 1.27 1.27)) hide)
     )
@@
     (property "Reference" "R27" (id 0) (at 184.15 48.26 90))
     (property "Value" "220" (id 1) (at 184.15 50.8 90))
-    (property "Footprint" "" (id 2) (at 184.15 55.753 90)
+    (property "Footprint" "Resistor_SMD:R_0603_1608Metric" (id 2) (at 184.15 55.753 90)
       (effects (font (size 1.27 1.27)) hide)
     )
@@
     (property "Reference" "R23" (id 0) (at 59.055 48.26 90))
     (property "Value" "220" (id 1) (at 59.055 50.8 90))
-    (property "Footprint" "" (id 2) (at 59.055 55.753 90)
-      (effects (font (size 1.27 1.27)) hide)
-    )
+    (property "Footprint" "Resistor_SMD:R_0603_1608Metric" (id 2) (at 59.055 55.753 90)
+      (effects (font (size 1.27 1.27)) hide)
+    )
