File: Relays_and_sensor.kicad_sch (KiCad schematic)
At the start: 29 parts, among them J4 Screw_Terminal_01x02, J5 Screw_Terminal_01x02, J6 Screw_Terminal_01x02, J7 Screw_Terminal_01x02, J8 Screw_Terminal_01x02, K1 1461103-1, K2 1461103-1, K3 1461103-1, K4 1461103-1, Q1 ZTX450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

Commit message: footprints
Parts:
- D1, D2, D3, D4: footprint (none) -> 1N4007G:DIOAD1036W78L470D235
- J4, J5, J6, J7, J8: footprint (none) -> TerminalBlock:TerminalBlock_bornier-2_P5.08mm
- K1, K2, K3, K4: footprint (none) -> Project_lic_footprints_AM:OJ_OJE
- Q1, Q2, Q3, Q4: footprint (none) -> eec:TO92250P510H770-3
Changed lines of the file:
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@@
       (effects (font (size 1.27 1.27)) (justify right))
     )
-    (property "Footprint" "" (id 2) (at 66.04 36.83 0)
+    (property "Footprint" "1N4007G:DIOAD1036W78L470D235" (id 2) (at 66.04 36.83 0)
       (effects (font (size 1.27 1.27)) (justify left bottom) hide)
     )
@@
       (effects (font (size 1.27 1.27)) (justify left))
     )
-    (property "Footprint" "" (id 2) (at 77.47 51.435 0)
+    (property "Footprint" "eec:TO92250P510H770-3" (id 2) (at 77.47 51.435 0)
       (effects (font (size 1.27 1.27)) hide)
     )
@@
       (effects (font (size 1.27 1.27)) (justify left))
     )
-    (property "Footprint" "" (id 2) (at 205.105 91.44 0)
+    (property "Footprint" "Project_lic_footprints_AM:OJ_OJE" (id 2) (at 205.105 91.44 0)
       (effects (font (size 1.27 1.27)) hide)
     )
@@
       (effects (font (size 1.27 1.27)) (justify left))
     )
-    (property "Footprint" "" (id 2) (at 246.38 35.56 0)
+    (property "Footprint" "TerminalBlock:TerminalBlock_bornier-2_P5.08mm" (id 2) (at 246.38 35.56 0)
       (effects (font (size 1.27 1.27)) hide)
     )
@@
       (effects (font (size 1.27 1.27)) (justify left))
     )
-    (property "Footprint" "" (id 2) (at 121.285 35.56 0)
+    (property "Footprint" "TerminalBlock:TerminalBlock_bornier-2_P5.08mm" (id 2) (at 121.285 35.56 0)
       (effects (font (size 1.27 1.27)) hide)
     )
@@
       (effects (font (size 1.27 1.27)) (justify right))
     )
-    (property "Footprint" "" (id 2) (at 66.04 86.36 0)
+    (property "Footprint" "1N4007G:DIOAD1036W78L470D235" (id 2) (at 66.04 86.36 0)
       (effects (font (size 1.27 1.27)) (justify left bottom) hide)
     )
@@
       (effects (font (size 1.27 1.27)) (justify left))
     )
-    (property "Footprint" "" (id 2) (at 246.38 85.09 0)
+    (property "Footprint" "TerminalBlock:TerminalBlock_bornier-2_P5.08mm" (id 2) (at 246.38 85.09 0)
       (effects (font (size 1.27 1.27)) hide)
     )
@@
       (effects (font (size 1.27 1.27)) (justify right))
     )
-    (property "Footprint" "" (id 2) (at 191.135 36.83 0)
+    (property "Footprint" "1N4007G:DIOAD1036W78L470D235" (id 2) (at 191.135 36.83 0)
       (effects (font (size 1.27 1.27)) (justify left bottom) hide)
     )
@@
       (effects (font (size 1.27 1.27)) (justify left))
     )
-    (property "Footprint" "" (id 2) (at 202.565 100.965 0)
+    (property "Footprint" "eec:TO92250P510H770-3" (id 2) (at 202.565 100.965 0)
       (effects (font (size 1.27 1.27)) hide)
     )
@@
       (effects (font (size 1.27 1.27)) (justify right))
     )
-    (property "Footprint" "" (id 2) (at 191.135 86.36 0)
+    (property "Footprint" "1N4007G:DIOAD1036W78L470D235" (id 2) (at 191.135 86.36 0)
       (effects (font (size 1.27 1.27)) (justify left bottom) hide)
     )
@@
       (effects (font (size 1.27 1.27)) (justify left))
     )
-    (property "Footprint" "" (id 2) (at 80.01 91.44 0)
+    (property "Footprint" "Project_lic_footprints_AM:OJ_OJE" (id 2) (at 80.01 91.44 0)
       (effects (font (size 1.27 1.27)) hide)
     )
@@
       (effects (font (size 1.27 1.27)) (justify left))
     )
-    (property "Footprint" "" (id 2) (at 121.285 85.09 0)
+    (property "Footprint" "TerminalBlock:TerminalBlock_bornier-2_P5.08mm" (id 2) (at 121.285 85.09 0)
       (effects (font (size 1.27 1.27)) hide)
     )
@@
       (effects (font (size 1.27 1.27)) (justify left))
     )
-    (property "Footprint" "" (id 2) (at 77.47 100.965 0)
+    (property "Footprint" "eec:TO92250P510H770-3" (id 2) (at 77.47 100.965 0)
       (effects (font (size 1.27 1.27)) hide)
     )
@@
       (effects (font (size 1.27 1.27)) (justify left))
     )
-    (property "Footprint" "" (id 2) (at 202.565 51.435 0)
+    (property "Footprint" "eec:TO92250P510H770-3" (id 2) (at 202.565 51.435 0)
       (effects (font (size 1.27 1.27)) hide)
     )
@@
       (effects (font (size 1.27 1.27)) (justify left))
     )
-    (property "Footprint" "" (id 2) (at 205.105 41.91 0)
+    (property "Footprint" "Project_lic_footprints_AM:OJ_OJE" (id 2) (at 205.105 41.91 0)
       (effects (font (size 1.27 1.27)) hide)
     )
@@
       (effects (font (size 1.27 1.27)) (justify right))
     )
-    (property "Footprint" "" (id 2) (at 64.135 170.18 0)
+    (property "Footprint" "TerminalBlock:TerminalBlock_bornier-2_P5.08mm" (id 2) (at 64.135 170.18 0)
       (effects (font (size 1.27 1.27)) hide)
     )
@@
       (effects (font (size 1.27 1.27)) (justify left))
     )
-    (property "Footprint" "" (id 2) (at 80.01 41.91 0)
-      (effects (font (size 1.27 1.27)) hide)
-    )
+    (property "Footprint" "Project_lic_footprints_AM:OJ_OJE" (id 2) (at 80.01 41.91 0)
+      (effects (font (size 1.27 1.27)) hide)
+    )

Commit message: PCB update
Parts:
- K1, K2, K3, K4: value 1461103-1 -> 6-1419128-4
Connections:
- net +24V: now also D1.C, D2.C, D3.C, D4.C, K1.2, K2.2, K3.2, K4.2, U3.10, U3.12, U3.14, U3.16
- net VDD: no longer D1.C, D2.C, D3.C, D4.C, K1.2, K2.2, K3.2, K4.2, U3.10, U3.12, U3.14, U3.16
Changed lines of the file:
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@@
     (effects (font (size 1.27 1.27)) (justify left))
-  )
-  (symbol (lib_id "power:VDD") (at 200.025 26.67 0) (unit 1)
-    (in_bom yes) (on_board yes) (fields_autoplaced)
-    (property "Reference" "#PWR053" (id 0) (at 200.025 30.48 0)
-      (effects (font (size 1.27 1.27)) hide)
-    )
-    (property "Value" "VDD" (id 1) (at 200.025 21.59 0))
-    (property "Footprint" "" (id 2) (at 200.025 26.67 0)
-      (effects (font (size 1.27 1.27)) hide)
-    )
-    (property "Datasheet" "" (id 3) (at 200.025 26.67 0)
-      (effects (font (size 1.27 1.27)) hide)
-    )
-    (pin "1")
   )
   (symbol (lib_id "power:VDD") (at 43.815 170.18 90) (unit 1)
@@
   )
   (symbol (lib_id "Project_lib_symbols_AM:1461103-1") (at 205.105 91.44 0) (unit 1)
-    (in_bom yes) (on_board yes) (fields_autoplaced)
+    (in_bom yes) (on_board yes)
     (property "Reference" "K4" (id 0) (at 227.33 85.0899 0)
       (effects (font (size 1.27 1.27)) (justify left))
     )
-    (property "Value" "1461103-1" (id 1) (at 227.33 87.6299 0)
+    (property "Value" "6-1419128-4" (id 1) (at 226.695 87.63 0)
       (effects (font (size 1.27 1.27)) (justify left))
     )
@@
     (pin "2")
   )
+  (symbol (lib_id "power:+24V") (at 200.025 26.67 0) (unit 1)
+    (in_bom yes) (on_board yes) (fields_autoplaced)
+    (property "Reference" "#PWR?" (id 0) (at 200.025 30.48 0)
+      (effects (font (size 1.27 1.27)) hide)
+    )
+    (property "Value" "+24V" (id 1) (at 200.025 21.59 0))
+    (property "Footprint" "" (id 2) (at 200.025 26.67 0)
+      (effects (font (size 1.27 1.27)) hide)
+    )
+    (property "Datasheet" "" (id 3) (at 200.025 26.67 0)
+      (effects (font (size 1.27 1.27)) hide)
+    )
+    (pin "1")
+  )
   (symbol (lib_id "Connector:Screw_Terminal_01x02") (at 121.285 35.56 0) (unit 1)
     (in_bom yes) (on_board yes)
@@
     (pin "1")
     (pin "2")
-  )
-  (symbol (lib_id "power:VDD") (at 200.025 76.2 0) (unit 1)
-    (in_bom yes) (on_board yes)
-    (property "Reference" "#PWR055" (id 0) (at 200.025 80.01 0)
-      (effects (font (size 1.27 1.27)) hide)
-    )
-    (property "Value" "VDD" (id 1) (at 200.025 71.755 0))
-    (property "Footprint" "" (id 2) (at 200.025 76.2 0)
-      (effects (font (size 1.27 1.27)) hide)
-    )
-    (property "Datasheet" "" (id 3) (at 200.025 76.2 0)
-      (effects (font (size 1.27 1.27)) hide)
-    )
-    (pin "1")
   )
   (symbol (lib_id "Isolator:LTV-844") (at 43.18 100.965 0) (unit 2)
@@
     (pin "9")
   )
+  (symbol (lib_id "power:+24V") (at 74.93 76.2 0) (unit 1)
+    (in_bom yes) (on_board yes) (fields_autoplaced)
+    (property "Reference" "#PWR?" (id 0) (at 74.93 80.01 0)
+      (effects (font (size 1.27 1.27)) hide)
+    )
+    (property "Value" "+24V" (id 1) (at 74.93 71.12 0))
+    (property "Footprint" "" (id 2) (at 74.93 76.2 0)
+      (effects (font (size 1.27 1.27)) hide)
+    )
+    (property "Datasheet" "" (id 3) (at 74.93 76.2 0)
+      (effects (font (size 1.27 1.27)) hide)
+    )
+    (pin "1")
+  )
   (symbol (lib_id "Device:R") (at 153.67 98.425 90) (unit 1)
     (in_bom yes) (on_board yes) (fields_autoplaced)
@@
     (pin "1")
   )
-  (symbol (lib_id "power:VDD") (at 74.93 26.67 0) (unit 1)
-    (in_bom yes) (on_board yes) (fields_autoplaced)
-    (property "Reference" "#PWR045" (id 0) (at 74.93 30.48 0)
-      (effects (font (size 1.27 1.27)) hide)
-    )
-    (property "Value" "VDD" (id 1) (at 74.93 21.59 0))
-    (property "Footprint" "" (id 2) (at 74.93 26.67 0)
-      (effects (font (size 1.27 1.27)) hide)
-    )
-    (property "Datasheet" "" (id 3) (at 74.93 26.67 0)
-      (effects (font (size 1.27 1.27)) hide)
-    )
-    (pin "1")
-  )
   (symbol (lib_id "power:GND") (at 153.035 63.5 0) (unit 1)
     (in_bom yes) (on_board yes) (fields_autoplaced)
@@
     )
     (property "Datasheet" "" (id 3) (at 200.025 63.5 0)
+      (effects (font (size 1.27 1.27)) hide)
+    )
+    (pin "1")
+  )
+  (symbol (lib_id "power:+24V") (at 74.93 26.67 0) (unit 1)
+    (in_bom yes) (on_board yes) (fields_autoplaced)
+    (property "Reference" "#PWR?" (id 0) (at 74.93 30.48 0)
+      (effects (font (size 1.27 1.27)) hide)
+    )
+    (property "Value" "+24V" (id 1) (at 74.93 21.59 0))
+    (property "Footprint" "" (id 2) (at 74.93 26.67 0)
+      (effects (font (size 1.27 1.27)) hide)
+    )
+    (property "Datasheet" "" (id 3) (at 74.93 26.67 0)
       (effects (font (size 1.27 1.27)) hide)
     )
@@
     (pin "1")
   )
-  (symbol (lib_id "Project_lib_symbols_AM:1461103-1") (at 80.01 91.44 0) (unit 1)
-    (in_bom yes) (on_board yes) (fields_autoplaced)
+  (symbol (lib_name "1461103-1_2") (lib_id "Project_lib_symbols_AM:1461103-1") (at 80.01 91.44 0) (unit 1)
+    (in_bom yes) (on_board yes)
     (property "Reference" "K2" (id 0) (at 102.235 85.0899 0)
       (effects (font (size 1.27 1.27)) (justify left))
     )
-    (property "Value" "1461103-1" (id 1) (at 102.235 87.6299 0)
+    (property "Value" "6-1419128-4" (id 1) (at 101.6 87.63 0)
       (effects (font (size 1.27 1.27)) (justify left))
     )
@@
     (pin "2")
   )
-  (symbol (lib_id "power:VDD") (at 74.93 76.2 0) (unit 1)
-    (in_bom yes) (on_board yes)
-    (property "Reference" "#PWR047" (id 0) (at 74.93 80.01 0)
-      (effects (font (size 1.27 1.27)) hide)
-    )
-    (property "Value" "VDD" (id 1) (at 74.93 72.39 0))
-    (property "Footprint" "" (id 2) (at 74.93 76.2 0)
-      (effects (font (size 1.27 1.27)) hide)
-    )
-    (property "Datasheet" "" (id 3) (at 74.93 76.2 0)
-      (effects (font (size 1.27 1.27)) hide)
-    )
-    (pin "1")
-  )
   (symbol (lib_id "power:+24V") (at 99.695 48.26 0) (unit 1)
     (in_bom yes) (on_board yes)
@@
     (pin "3")
   )
-  (symbol (lib_id "Project_lib_symbols_AM:1461103-1") (at 205.105 41.91 0) (unit 1)
+  (symbol (lib_name "1461103-1_3") (lib_id "Project_lib_symbols_AM:1461103-1") (at 205.105 41.91 0) (unit 1)
     (in_bom yes) (on_board yes) (fields_autoplaced)
     (property "Reference" "K3" (id 0) (at 227.33 35.5599 0)
       (effects (font (size 1.27 1.27)) (justify left))
     )
-    (property "Value" "1461103-1" (id 1) (at 227.33 38.0999 0)
+    (property "Value" "6-1419128-4" (id 1) (at 227.33 38.0999 0)
       (effects (font (size 1.27 1.27)) (justify left))
     )
@@
     )
     (property "Datasheet" "" (id 3) (at 241.3 43.815 0)
+      (effects (font (size 1.27 1.27)) hide)
+    )
+    (pin "1")
+  )
+  (symbol (lib_id "power:+24V") (at 200.025 76.2 0) (unit 1)
+    (in_bom yes) (on_board yes) (fields_autoplaced)
+    (property "Reference" "#PWR?" (id 0) (at 200.025 80.01 0)
+      (effects (font (size 1.27 1.27)) hide)
+    )
+    (property "Value" "+24V" (id 1) (at 200.025 71.12 0))
+    (property "Footprint" "" (id 2) (at 200.025 76.2 0)
+      (effects (font (size 1.27 1.27)) hide)
+    )
+    (property "Datasheet" "" (id 3) (at 200.025 76.2 0)
       (effects (font (size 1.27 1.27)) hide)
     )
@@
     (pin "1")
   )
-  (symbol (lib_id "Project_lib_symbols_AM:1461103-1") (at 80.01 41.91 0) (unit 1)
-    (in_bom yes) (on_board yes) (fields_autoplaced)
+  (symbol (lib_name "1461103-1_1") (lib_id "Project_lib_symbols_AM:1461103-1") (at 80.01 41.91 0) (unit 1)
+    (in_bom yes) (on_board yes)
     (property "Reference" "K1" (id 0) (at 102.235 35.5599 0)
       (effects (font (size 1.27 1.27)) (justify left))
     )
-    (property "Value" "1461103-1" (id 1) (at 102.235 38.0999 0)
-      (effects (font (size 1.27 1.27)) (justify left))
-    )
+    (property "Value" "6-1419128-4" (id 1) (at 101.6 38.1 0)
+      (effects (font (size 1.27 1.27)) (justify left))
+    )
